File: kicad/control_units/classic/led/led.kicad_sch (KiCad schematic)
At the start: 0 parts

Commit message: feat: created LED board schematic for the Classic control unit (8 LEDs) using 74HC595 shift register, measurements needed for actual PCB
Parts:
- added C1: 100n, symbol Device:C
- added D1, D2, D3, D4, D5, D6, D7, D8: LED, symbol Device:LED
- added J1: Conn_01x03, symbol Connector_Generic:Conn_01x03
- added Q1, Q2, Q3, Q4, Q5, Q6, Q7, Q8: BC547, Package_TO_SOT_THT:TO-92_Inline, symbol Transistor_BJT:BC547
- added R1, R12, R17, R18, R23, R24, R6, R9: 180, symbol Device:R
- added R10, R13, R14, R19, R20, R3, R4, R7: 1.3k, symbol Device:R
- added R11, R15, R16, R2, R21, R22, R5, R8: 47k, symbol Device:R
- added U1: 74HC595, symbol 74xx:74HC595
Connections:
- new net: Q5.2 (B), R13.2, R15.1
- new net: J1.1 (Pin_1), U1.14 (SER)
- new net: J1.2 (Pin_2), U1.11 (SRCLK)
- new net: J1.3 (Pin_3), U1.12 (RCLK)
- new net: Q4.2 (B), R10.2, R11.1
- new net: Q1.2 (B), R2.1, R3.2
- new net: D1.1 (K), Q1.1 (C)
- new net: D5.1 (K), Q5.1 (C)
- new net: D5.2 (A), R17.2
- new net: D7.1 (K), Q7.1 (C)
- new net: Q7.2 (B), R19.2, R21.1
- new net: D8.1 (K), Q8.1 (C)
- new net: D8.2 (A), R24.2
- new net: D4.1 (K), Q4.1 (C)
- new net: D3.1 (K), Q3.1 (C)
- new net: Q3.2 (B), R7.2, R8.1
- new net: Q8.2 (B), R20.2, R22.1
- new net: D7.2 (A), R23.2
- new net: D1.2 (A), R1.2
- new net: D6.2 (A), R18.2
- new net: Q2.2 (B), R4.2, R5.1
- new net: D4.2 (A), R12.2
- new net: D6.1 (K), Q6.1 (C)
- new net: Q6.2 (B), R14.2, R16.1
- new net: D2.2 (A), R6.2
- new net: D3.2 (A), R9.2
- new net: D2.1 (K), Q2.1 (C)
- new net +3V3: C1.1, R1.1, R12.1, R17.1, R18.1, R23.1, R24.1, R6.1, R9.1, U1.10 (~{SRCLR}), U1.16 (VCC)
- new net GND: C1.2, Q1.3 (E), Q2.3 (E), Q3.3 (E), Q4.3 (E), Q5.3 (E), Q6.3 (E), Q7.3 (E), Q8.3 (E), R11.2, R15.2, R16.2, R2.2, R21.2, R22.2, R5.2, R8.2, U1.13 (~{OE}), U1.8 (GND)
- new net LED_A1: R3.1, U1.15 (QA)
- new net LED_A2: R7.1, U1.1 (QB)
- new net LED_A3: R13.1, U1.2 (QC)
- new net LED_A4: R14.1, U1.3 (QD)
- new net LED_B1: R4.1, U1.4 (QE)
- new net LED_B2: R10.1, U1.5 (QF)
- new net LED_B3: R19.1, U1.6 (QG)
- new net LED_B4: R20.1, U1.7 (QH)
- no-connect marks 0 -> 1

Commit message: More stuff for Classic control unit
Parts:
- removed C1: 100n, symbol Device:C
- removed J1: Conn_01x03, symbol Connector_Generic:Conn_01x03
- added C2: 100n, symbol Device:C
- added J2: Conn_01x05, symbol Connector_Generic:Conn_01x05
Connections:
- net +3V3: now also C2.1, J2.1 (Pin_1)
- net GND: now also C2.2, J2.5 (Pin_5)
- net at U1.14 (SER): now also J2.2 (Pin_2)
- net at U1.11 (SRCLK): now also J2.3 (Pin_3)
- net at U1.12 (RCLK): now also J2.4 (Pin_4)

Commit message: feat: Added connector schematics and fixed some other connectors in other schematics
Connections:
- net +3V3: now also J2.5 (Pin_5); no longer J2.1 (Pin_1)
- net GND: now also J2.1 (Pin_1); no longer J2.5 (Pin_5)
- net at J2.2 (Pin_2): now also U1.12 (RCLK); no longer U1.14 (SER)
- net at J2.4 (Pin_4): now also U1.14 (SER); no longer U1.12 (RCLK)
Changed lines of the file:
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@@
 	(wire
 		(pts
-			(xy 40.64 78.74) (xy 40.64 97.79)
-		)
-		(stroke
-			(width 0)
-			(type default)
-		)
-	)
-	(wire
-		(pts
 			(xy 266.7 132.08) (xy 266.7 129.54)
 		)
@@
 	(wire
 		(pts
-			(xy 38.1 78.74) (xy 38.1 92.71)
+			(xy 40.64 78.74) (xy 40.64 97.79)
 		)
 		(stroke
@@
 	(wire
 		(pts
+			(xy 38.1 78.74) (xy 38.1 105.41)
+		)
+		(stroke
+			(width 0)
+			(type default)
+		)
+	)
+	(wire
+		(pts
 			(xy 148.59 166.37) (xy 152.4 166.37)
 		)
@@
 	(wire
 		(pts
-			(xy 43.18 78.74) (xy 43.18 105.41)
+			(xy 38.1 105.41) (xy 54.61 105.41)
+		)
+		(stroke
+			(width 0)
+			(type default)
+		)
+	)
+	(wire
+		(pts
+			(xy 43.18 92.71) (xy 54.61 92.71)
 		)
 		(stroke
@@
 	(wire
 		(pts
-			(xy 95.25 78.74) (xy 95.25 77.47)
+			(xy 40.64 97.79) (xy 54.61 97.79)
 		)
 		(stroke
@@
 	(wire
 		(pts
-			(xy 40.64 97.79) (xy 54.61 97.79)
+			(xy 95.25 78.74) (xy 95.25 77.47)
 		)
 		(stroke
@@
 	(wire
 		(pts
-			(xy 54.61 120.65) (xy 64.77 120.65)
+			(xy 43.18 78.74) (xy 43.18 92.71)
 		)
 		(stroke
@@
 	(wire
 		(pts
-			(xy 201.93 82.55) (xy 204.47 82.55)
+			(xy 54.61 120.65) (xy 64.77 120.65)
 		)
 		(stroke
@@
 	(wire
 		(pts
-			(xy 74.93 97.79) (xy 77.47 97.79)
+			(xy 201.93 82.55) (xy 204.47 82.55)
 		)
 		(stroke
@@
 	(wire
 		(pts
-			(xy 160.02 48.26) (xy 160.02 45.72)
+			(xy 74.93 97.79) (xy 77.47 97.79)
 		)
 		(stroke
@@
 	(wire
 		(pts
-			(xy 43.18 105.41) (xy 54.61 105.41)
+			(xy 160.02 48.26) (xy 160.02 45.72)
 		)
 		(stroke
@@
 	(wire
 		(pts
-			(xy 38.1 92.71) (xy 54.61 92.71)
-		)
-		(stroke
-			(width 0)
-			(type default)
-		)
-	)
-	(wire
-		(pts
 			(xy 74.93 107.95) (xy 77.47 107.95)
 		)
@@
 	)
 	(symbol
-		(lib_id "power:+3V3")
-		(at 35.56 78.74 90)
-		(unit 1)
-		(body_style 1)
-		(exclude_from_sim no)
-		(in_bom yes)
-		(on_board yes)
-		(in_pos_files yes)
-		(dnp no)
-		(fields_autoplaced yes)
-		(property "Reference" "#PWR027"
-			(at 39.37 78.74 0)
-			(hide yes)
-			(show_name no)
-			(do_not_autoplace no)
-			(effects
-				(font
-					(size 1.27 1.27)
-				)
-			)
-		)
-		(property "Value" "+3V3"
-			(at 31.75 78.7399 90)
-			(show_name no)
-			(do_not_autoplace no)
-			(effects
-				(font
-					(size 1.27 1.27)
-				)
-				(justify left)
-			)
-		)
-		(property "Footprint" ""
-			(at 35.56 78.74 0)
-			(hide yes)
-			(show_name no)
-			(do_not_autoplace no)
-			(effects
-				(font
-					(size 1.27 1.27)
-				)
-			)
-		)
-		(property "Datasheet" ""
-			(at 35.56 78.74 0)
-			(hide yes)
-			(show_name no)
-			(do_not_autoplace no)
-			(effects
-				(font
-					(size 1.27 1.27)
-				)
-			)
-		)
-		(property "Description" "Power symbol creates a global label with name \"+3V3\""
-			(at 35.56 78.74 0)
-			(hide yes)
-			(show_name no)
-			(do_not_autoplace no)
-			(effects
-				(font
-					(size 1.27 1.27)
-				)
-			)
-		)
-		(pin "1"
-		)
-		(instances
-			(project "led"
-				(path "/7c3be559-9ecd-4615-b96b-4e36dbf74286"
-					(reference "#PWR027")
-					(unit 1)
-				)
-			)
-		)
-	)
-	(symbol
 		(lib_id "Device:R")
 		(at 160.02 24.13 0)
@@
 	(symbol
 		(lib_id "power:GND")
+		(at 35.56 78.74 0)
+		(unit 1)
+		(body_style 1)
+		(exclude_from_sim no)
+		(in_bom yes)
+		(on_board yes)
+		(in_pos_files yes)
+		(dnp no)
+		(fields_autoplaced yes)
+		(property "Reference" "#PWR028"
+			(at 35.56 85.09 0)
+			(hide yes)
+			(show_name no)
+			(do_not_autoplace no)
+			(effects
+				(font
+					(size 1.27 1.27)
+				)
+			)
+		)
+		(property "Value" "GND"
+			(at 35.56 83.82 0)
+			(show_name no)
+			(do_not_autoplace no)
+			(effects
+				(font
+					(size 1.27 1.27)
+				)
+			)
+		)
+		(property "Footprint" ""
+			(at 35.56 78.74 0)
+			(hide yes)
+			(show_name no)
+			(do_not_autoplace no)
+			(effects
+				(font
+					(size 1.27 1.27)
+				)
+			)
+		)
+		(property "Datasheet" ""
+			(at 35.56 78.74 0)
+			(hide yes)
+			(show_name no)
+			(do_not_autoplace no)
+			(effects
+				(font
+					(size 1.27 1.27)
+				)
+			)
+		)
+		(property "Description" "Power symbol creates a global label with name \"GND\" , ground"
+			(at 35.56 78.74 0)
+			(hide yes)
+			(show_name no)
+			(do_not_autoplace no)
+			(effects
+				(font
+					(size 1.27 1.27)
+				)
+			)
+		)
+		(pin "1"
+		)
+		(instances
+			(project "led"
+				(path "/7c3be559-9ecd-4615-b96b-4e36dbf74286"
+					(reference "#PWR028")
+					(unit 1)
+				)
+			)
+		)
+	)
+	(symbol
+		(lib_id "power:GND")
 		(at 148.59 48.26 0)
 		(unit 1)
@@
 	(symbol
 		(lib_id "power:GND")
-		(at 45.72 78.74 90)
+		(at 148.59 173.99 0)
 		(unit 1)
 		(body_style 1)
@@
 		(dnp no)
 		(fields_autoplaced yes)
-		(property "Reference" "#PWR028"
-			(at 52.07 78.74 0)
+		(property "Reference" "#PWR014"
+			(at 148.59 180.34 0)
 			(hide yes)
 			(show_name no)
@@
 		)
 		(property "Value" "GND"
-			(at 49.53 78.7399 90)
+			(at 148.59 179.07 0)
 			(show_name no)
 			(do_not_autoplace no)
@@
 					(size 1.27 1.27)
 				)
-				(justify right)
 			)
 		)
 		(property "Footprint" ""
-			(at 45.72 78.74 0)
+			(at 148.59 173.99 0)
 			(hide yes)
 			(show_name no)
@@
 		)
 		(property "Datasheet" ""
-			(at 45.72 78.74 0)
+			(at 148.59 173.99 0)
 			(hide yes)
 			(show_name no)
@@
 		)
 		(property "Description" "Power symbol creates a global label with name \"GND\" , ground"
-			(at 45.72 78.74 0)
+			(at 148.59 173.99 0)
 			(hide yes)
 			(show_name no)
@@
 			(project "led"
 				(path "/7c3be559-9ecd-4615-b96b-4e36dbf74286"
-					(reference "#PWR028")
+					(reference "#PWR014")
 					(unit 1)
 				)
@@
 	)
 	(symbol
-		(lib_id "power:GND")
-		(at 148.59 173.99 0)
+		(lib_id "power:+3V3")
+		(at 45.72 78.74 180)
 		(unit 1)
 		(body_style 1)
@@
 		(dnp no)
 		(fields_autoplaced yes)
-		(property "Reference" "#PWR014"
-			(at 148.59 180.34 0)
+		(property "Reference" "#PWR027"
+			(at 45.72 74.93 0)
 			(hide yes)
 			(show_name no)
@@
 			)
 		)
-		(property "Value" "GND"
-			(at 148.59 179.07 0)
+		(property "Value" "+3V3"
+			(at 45.72 83.82 0)
 			(show_name no)
 			(do_not_autoplace no)
@@
 		)
 		(property "Footprint" ""
-			(at 148.59 173.99 0)
+			(at 45.72 78.74 0)
 			(hide yes)
 			(show_name no)
@@
 		)
 		(property "Datasheet" ""
-			(at 148.59 173.99 0)
+			(at 45.72 78.74 0)
 			(hide yes)
 			(show_name no)
@@
 			)
 		)
-		(property "Description" "Power symbol creates a global label with name \"GND\" , ground"
-			(at 148.59 173.99 0)
+		(property "Description" "Power symbol creates a global label with name \"+3V3\""
+			(at 45.72 78.74 0)
 			(hide yes)
 			(show_name no)
@@
 			(project "led"
 				(path "/7c3be559-9ecd-4615-b96b-4e36dbf74286"
-					(reference "#PWR014")
+					(reference "#PWR027")
 					(unit 1)
 				)

Commit message: feat: Should be able to footprint and route some prototype boards to see if I'm not totally off-base here
Parts:
- removed C2: 100n, symbol Device:C
- added C1: 100n, symbol Device:C
Connections:
- net +3V3: now also C1.1
- net GND: now also C1.2

Commit message: feat: Should now be able to order some prototype PCBs to see if this whole thing actually works; note to self, buy some DIP sockets
Parts:
- C1: footprint (none) -> Capacitor_THT:C_Disc_D5.0mm_W2.5mm_P2.50mm
- D1, D2, D3, D4, D5, D6, D7, D8: footprint (none) -> LED_THT:LED_D5.0mm
- J2: footprint (none) -> Connector_PinSocket_2.54mm:PinSocket_1x05_P2.54mm_Vertical
- R1, R10, R11, R12, R13, R14, R15, R16, R17, R18, R19, R2, R20, R21, R22, R23, R24, R3, R4, R5, R6, R7, R8, R9: footprint (none) -> Resistor_THT:R_Axial_DIN0207_L6.3mm_D2.5mm_P7.62mm_Horizontal
- U1: footprint (none) -> Package_DIP:DIP-16_W7.62mm
